File: Kicad Files/Typewriter Keyboard Controller.kicad_pcb (KiCad board)
At the start: 2 copper layers, 88.9 x 76.2 mm, 40 parts, among them J1 USB_mini_micro_B, P1 CONN_01X08, P2 CONN_01X08, SW1 SW_PUSH, U1 ATMEGA32U4, X1 XTAL_GND

Commit message: Make mouting holes smaller
Parts:
- removed the REF** at (108.0, 120.7)
- removed the REF** at (184.2, 101.6)
- removed the REF** at (113.0, 57.1)
- added REF**: MountingHole_3mm, Mounting_Holes:MountingHole_3mm, F.Cu at (184.2, 101.6)
- added REF**: MountingHole_3mm, Mounting_Holes:MountingHole_3mm, F.Cu at (113.0, 57.1)
- added REF**: MountingHole_3mm, Mounting_Holes:MountingHole_3mm, F.Cu at (108.0, 120.7)
Changed lines of the file:
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@@
 (kicad_pcb (version 4) (host pcbnew 4.0.2+dfsg1-stable)
   (general
-    (links 90)
+    (links 0)
     (no_connects 0)
-    (area 101.524999 50.724999 190.575001 127.075001)
+    (area 100.460714 47.971 191.639286 128.62524)
     (thickness 1.6)
     (drawings 21)
@@
       (outputformat 1)
       (mirror false)
-      (drillshape 1)
+      (drillshape 0)
       (scaleselection 1)
       (outputdirectory ""))
@@
       (rotate (xyz 0 0 90))
     )
-  )
-  (module Mounting_Holes:MountingHole_5mm (layer F.Cu)
-    (at 107.95 120.65)
-    (descr "Mounting hole, Befestigungsbohrung, 5mm, No Annular, Kein Restring,")
-    (tags "Mounting hole, Befestigungsbohrung, 5mm, No Annular, Kein Restring,")
-    (fp_text reference REF** (at 0 -6.49986) (layer F.SilkS) hide
-      (effects (font (size 1 1) (thickness 0.15)))
-    )
-    (fp_text value MountingHole_5mm (at 0 7.00024) (layer F.Fab) hide
-      (effects (font (size 1 1) (thickness 0.15)))
-    )
-    (fp_circle (center 0 0) (end 5 0) (layer Cmts.User) (width 0.381))
-    (pad 1 thru_hole circle (at 0 0) (size 5 5) (drill 5) (layers))
-  )
-  (module Mounting_Holes:MountingHole_5mm (layer F.Cu)
-    (at 184.15 101.6)
-    (descr "Mounting hole, Befestigungsbohrung, 5mm, No Annular, Kein Restring,")
-    (tags "Mounting hole, Befestigungsbohrung, 5mm, No Annular, Kein Restring,")
-    (fp_text reference REF** (at 0 -6.49986) (layer F.SilkS) hide
-      (effects (font (size 1 1) (thickness 0.15)))
-    )
-    (fp_text value MountingHole_5mm (at 0 7.00024) (layer F.Fab) hide
-      (effects (font (size 1 1) (thickness 0.15)))
-    )
-    (fp_circle (center 0 0) (end 5 0) (layer Cmts.User) (width 0.381))
-    (pad 1 thru_hole circle (at 0 0) (size 5 5) (drill 5) (layers))
-  )
-  (module Mounting_Holes:MountingHole_5mm (layer F.Cu)
-    (at 113.03 57.15)
-    (descr "Mounting hole, Befestigungsbohrung, 5mm, No Annular, Kein Restring,")
-    (tags "Mounting hole, Befestigungsbohrung, 5mm, No Annular, Kein Restring,")
-    (fp_text reference REF** (at 0 -6.49986) (layer F.SilkS) hide
-      (effects (font (size 1 1) (thickness 0.15)))
-    )
-    (fp_text value MountingHole_5mm (at 0 7.00024) (layer F.Fab) hide
-      (effects (font (size 1 1) (thickness 0.15)))
-    )
-    (fp_circle (center 0 0) (end 5 0) (layer Cmts.User) (width 0.381))
-    (pad 1 thru_hole circle (at 0 0) (size 5 5) (drill 5) (layers))
   )
   (module "Lynx:Lynx medium" (layer F.Cu)
@@
       (xy 2.579248 -1.867447) (xy 2.625684 -1.868766) (xy 2.67841 -1.862378)) (layer F.SilkS) (width 0.01))
   )
+  (module Mounting_Holes:MountingHole_3mm (layer F.Cu)
+    (at 184.15 101.6)
+    (descr "Mounting hole, Befestigungsbohrung, 3mm, No Annular, Kein Restring,")
+    (tags "Mounting hole, Befestigungsbohrung, 3mm, No Annular, Kein Restring,")
+    (fp_text reference REF** (at 0 -4.0005) (layer F.SilkS) hide
+      (effects (font (size 1 1) (thickness 0.15)))
+    )
+    (fp_text value MountingHole_3mm (at 1.00076 5.00126) (layer F.Fab) hide
+      (effects (font (size 1 1) (thickness 0.15)))
+    )
+    (fp_circle (center 0 0) (end 3 0) (layer Cmts.User) (width 0.381))
+    (pad 1 thru_hole circle (at 0 0) (size 3 3) (drill 3) (layers))
+  )
+  (module Mounting_Holes:MountingHole_3mm (layer F.Cu)
+    (at 113.03 57.15)
+    (descr "Mounting hole, Befestigungsbohrung, 3mm, No Annular, Kein Restring,")
+    (tags "Mounting hole, Befestigungsbohrung, 3mm, No Annular, Kein Restring,")
+    (fp_text reference REF** (at 0 -4.0005) (layer F.SilkS) hide
+      (effects (font (size 1 1) (thickness 0.15)))
+    )
+    (fp_text value MountingHole_3mm (at 1.00076 5.00126) (layer F.Fab) hide
+      (effects (font (size 1 1) (thickness 0.15)))
+    )
+    (fp_circle (center 0 0) (end 3 0) (layer Cmts.User) (width 0.381))
+    (pad 1 thru_hole circle (at 0 0) (size 3 3) (drill 3) (layers))
+  )
+  (module Mounting_Holes:MountingHole_3mm (layer F.Cu)
+    (at 107.95 120.65)
+    (descr "Mounting hole, Befestigungsbohrung, 3mm, No Annular, Kein Restring,")
+    (tags "Mounting hole, Befestigungsbohrung, 3mm, No Annular, Kein Restring,")
+    (fp_text reference REF** (at 0 -4.0005) (layer F.SilkS) hide
+      (effects (font (size 1 1) (thickness 0.15)))
+    )
+    (fp_text value MountingHole_3mm (at 1.00076 5.00126) (layer F.Fab) hide
+      (effects (font (size 1 1) (thickness 0.15)))
+    )
+    (fp_circle (center 0 0) (end 3 0) (layer Cmts.User) (width 0.381))
+    (pad 1 thru_hole circle (at 0 0) (size 3 3) (drill 3) (layers))
+  )
   (gr_circle (center 158.75 98.425) (end 158.75 97.79) (layer F.SilkS) (width 0.2))
