File: Kicad Files/Typewriter Keyboard Controller.sch (KiCad schematic (older format))
At the start: 36 parts, among them J1 USB_mini_micro_B, P1 CONN_01X08, P2 CONN_01X08, SW1 SW_PUSH, U1 ATMEGA32U4, X1 XTAL_GND

Commit message: update to KiCad 5
Parts:
- C1, C2, C3, C4, C5, C6, C7, C8: symbol C -> Typewriter-Keyboard-Controller-rescue:C
- J1: symbol USB_mini_micro_B -> keyboard_parts:USB_mini_micro_B
- LED1, LED2, LED3, LED4, LED5, LED6, LED7, LED8, LED9: symbol LED -> Typewriter-Keyboard-Controller-rescue:LED
- P1, P2: symbol CONN_01X08 -> Typewriter-Keyboard-Controller-rescue:CONN_01X08
- R1, R10, R11, R12, R13, R2, R3, R4, R5, R6, R7, R8, R9: symbol R -> Typewriter-Keyboard-Controller-rescue:R
- SW1: symbol SW_PUSH -> keyboard_parts:SW_PUSH
- U1: symbol ATMEGA32U4 -> keyboard_parts:ATMEGA32U4
- X1: symbol XTAL_GND -> keyboard_parts:XTAL_GND
